File: PCB-EAGLE/OsuKB.sch (EAGLE design)
At the start: 72 parts, among them X1 USB-MINIB-5PIN

Commit message: ed sh na
Parts:
- R10: value (none) -> 10k
- R13, R14: value (none) -> 1k
- S1.1, S2.1: value MP5 -> MP9R-1
- VD1, VD2: value (none) -> 3v6
Other:
- moved on the sheet: JP7, R13, R14
